File: NoU3-MotorDriver.kicad_sch (KiCad schematic)
At the start: 6 parts, among them J2 Screw_Terminal_01x02, J3 Screw_Terminal_01x02, U1 HR8833

Commit message: Updated to KiCAD 10.0
Parts:
- J2, J3: LCSC C8404 -> C557646

Commit message: cleaned up JSTs on motor driver sheet
Parts:
- added J1: JST SR/SZ, AlfredoFootprints:JST_SH_1x06_Vertical, symbol Connector_Generic:Conn_01x06
Connections:
- net +3V3: now also J1.4 (Pin_4)
- net GND: now also J1.1 (Pin_1)
- net Aout1: no longer names the net of J2.2 (Pin_2), U1.2 (AOUT1)
- net Aout1: now also J1.6 (Pin_6)
- net Aout2: no longer names the net of J2.1 (Pin_1), U1.4 (AOUT2)
- net Aout2: now also J1.5 (Pin_5)
- new net ENC_A: J1.3 (Pin_3)
- new net ENC_B: J1.2 (Pin_2)

Commit message: first push with NoU3.7 features
Parts:
- added J20: JST SR/SZ, AlfredoFootprints:JST_SH_1x06_Vertical, symbol Connector_Generic:Conn_01x06
- added R29, R33: 100mR, Resistor_SMD:R_0805_2012Metric, symbol Device:R
Connections:
- net +3V3: now also J20.4 (Pin_4)
- net GND: now also J20.1 (Pin_1), R29.2, R33.2; no longer U1.3 (AISEN), U1.6 (BISEN)
- net Bout1: no longer names the net of J3.1 (Pin_1), U1.7 (BOUT1)
- net Bout1: now also J20.6 (Pin_6)
- net Bout2: no longer names the net of J3.2 (Pin_2), U1.5 (BOUT2)
- net Bout2: now also J20.5 (Pin_5)
- net ENC_A renamed ENC_A1
- net ENC_B renamed ENC_B1
- new net AISEN: R33.1, U1.3 (AISEN)
- new net BISEN: R29.1, U1.6 (BISEN)
- new net ENC_A2: J20.3 (Pin_3)
- new net ENC_B2: J20.2 (Pin_2)

Commit message: PY32F030K28U6TR motor controller chip
Parts:
- renumbered J1 to J19, J20 to J4, J2 to J5, J3 to J6
Connections:
- net AIN1 renamed MOTOR_SIGNAL_1A
- net AIN2 renamed MOTOR_SIGNAL_1B
- net AISEN renamed SENSEI_1
- net BIN1 renamed MOTOR_SIGNAL_2B
- net BIN2 renamed MOTOR_SIGNAL_2A
- net BISEN renamed SENSEI_2
- net ENC_A1 renamed ENCODER_1A
- net ENC_A2 renamed ENCODER_2A
- net ENC_B1 renamed ENCODER_1B
- net ENC_B2 renamed ENCODER_2B
Other:
- moved on the sheet: R29, R33

Commit message: motor driver footprints
Parts:
- added R23, R37: 1K, Resistor_SMD:R_0402_1005Metric, symbol Device:R
Connections:
- net SENSEI_1: now also R23.2; no longer R33.1, U1.3 (AISEN)
- net SENSEI_2: now also R37.2; no longer R29.1, U1.6 (BISEN)
- net at J5.1 (Pin_1), U1.4 (AOUT2): now also J19.6 (Pin_6); no longer J19.5 (Pin_5)
- net at J5.2 (Pin_2), U1.2 (AOUT1): now also J19.5 (Pin_5); no longer J19.6 (Pin_6)
- new net: R29.1, R37.1, U1.6 (BISEN)
- new net: R23.1, R33.1, U1.3 (AISEN)
