File: NoU3.kicad_pcb (KiCad board)
At the start: 4 copper layers, 46 x 56 mm, 149 parts, among them J1 JST SR/SZ, J10 JST SR/SZ, J11 Screw_Terminal_01x02, J12 Screw_Terminal_01x02, J13 JST SR/SZ, J14 RFANT3216120A5T, J15 Barrel_Jack, J16 VIN, J17 JST SR/SZ, J18 GND, J19 JST SR/SZ, J2 Screw_Terminal_01x02, J20 JST SR/SZ, J3 Screw_Terminal_01x02, J4 JST SR/SZ, J5 Screw_Terminal_01x02, J6 Screw_Terminal_01x02, J7 JST SR/SZ, J8 Screw_Terminal_01x02, J9 Screw_Terminal_01x02, Q2 AONR21357, SW1 reset, SW2 boot, U1 HR8833, U10 PY32F030K28U6TR, U11 Qwiic1, U14 PY32F030K28U6TR, U15 SY8113BADC, U16 SY8113BADC, U17 USB_C_Receptacle, U18 ServoPorts_2x3, U19 ServoPorts_2x3, U2 ESP32-S3FN8, U26 LSM6DS3TR-C, U3 Crystal_ESP32, U4 HR8833, U5 HR8833, U6 HR8833, U7 ServoPorts_2x3, U8 5.8 ZSPT, U9 USBLC6-2P6

Commit message: motor driver footprints
Parts:
- removed the G*** at (-10.9, 13.8)
- removed R38, R39, R42, R43: 1K, Resistor_SMD:R_0402_1005Metric
- added C43: 220uF, AlfredoFootprints:CP_Elec_6.3x7.7_slim, F.Cu at (-4.40, -12.2)
- added R44: 1K, Resistor_SMD:R_0402_1005Metric, F.Cu at (-58.0, 27.3)
- added R45: 1K, Resistor_SMD:R_0402_1005Metric, F.Cu at (-58.0, 29.3)
- added R48: 1K, Resistor_SMD:R_0402_1005Metric, F.Cu at (-59.3, -36.2)
- added R49: 1K, Resistor_SMD:R_0402_1005Metric, F.Cu at (-55.9, -37.0)
- C11, C12, C13, R15, R16, U6: moved to B.Cu
- C16, C20, C42: footprint Capacitor_SMD:CP_Elec_6.3x7.7 -> AlfredoFootprints:CP_Elec_6.3x7.7_slim
- TP1, TP2, TP20, TP3: moved to F.Cu
- moved U6 105.4 mm to (40.2, -3.50), turned to -90 degrees
- moved C12 102.3 mm to (41.1, 0.88), turned to 0 degrees
- moved C13 98.6 mm to (39.3, 0.88), turned to 0 degrees
- moved U9 80.3 mm to (83.3, -1.84)
- moved C42 80.2 mm to (48.2, -24.1), turned to 180 degrees
- moved C15 72.8 mm to (86.8, 1.18)
- moved R26 72.8 mm to (85.0, 2.08)
- moved D2 72.8 mm to (82.2, 1.88)
- moved R27 72.8 mm to (86.8, 2.08)
- moved C16 68.2 mm to (57.0, -24.1), turned to 0 degrees
- moved U5 67.5 mm to (4.80, 11.9), turned to 180 degrees
- moved C9 59.9 mm to (0.44, 11.0), turned to 90 degrees
- moved C14 59.7 mm to (58.2, -53.8)
- moved C10 57.7 mm to (0.44, 12.8), turned to 90 degrees
- moved C1 48.1 mm to (35.9, -54.6)
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Connections:
- C19 pad 1: Net-(U10-PA0/ADC_IN0) -> /MotorSystem/MotorDriver-1/SENSEI_1
- C41 pad 1: Net-(U10-PA1/ADC_IN1) -> /MotorSystem/MotorDriver-1/SENSEI_2
- C44 pad 1: Net-(U10-PA2/ADC_IN2) -> /MotorSystem/MotorDriver-4/SENSEI_1
- C45 pad 1: Net-(U10-PA3/ADC_IN3) -> /MotorSystem/MotorDriver-4/SENSEI_2
- C49 pad 1: Net-(U14-PA0/ADC_IN0) -> /MotorSystem/MotorDriver-3/SENSEI_1
- C50 pad 1: Net-(U14-PA1/ADC_IN1) -> /MotorSystem/MotorDriver-3/SENSEI_2
- C51 pad 1: Net-(U14-PA2/ADC_IN2) -> /MotorSystem/MotorDriver-2/SENSEI_1
- C52 pad 1: Net-(U14-PA3/ADC_IN3) -> /MotorSystem/MotorDriver-2/SENSEI_2
- J11 pad 1: Net-(J10-Pin_5) -> Net-(J10-Pin_6)
- J11 pad 2: Net-(J10-Pin_6) -> Net-(J10-Pin_5)
- J2 pad 1: Net-(J1-Pin_5) -> Net-(J1-Pin_6)
- J2 pad 2: Net-(J1-Pin_6) -> Net-(J1-Pin_5)
- J5 pad 1: Net-(J19-Pin_5) -> Net-(J19-Pin_6)
- J5 pad 2: Net-(J19-Pin_6) -> Net-(J19-Pin_5)
- J8 pad 1: Net-(J7-Pin_5) -> Net-(J7-Pin_6)
- J8 pad 2: Net-(J7-Pin_6) -> Net-(J7-Pin_5)
- R23 pad 1: /MotorSystem/MotorDriver-1/SENSEI_1 -> Net-(U1-AISEN)
- R23 pad 2: Net-(U10-PA0/ADC_IN0) -> /MotorSystem/MotorDriver-1/SENSEI_1
- R29 pad 1: /MotorSystem/MotorDriver-1/SENSEI_2 -> Net-(U1-BISEN)
- R30 pad 1: /MotorSystem/MotorDriver-2/SENSEI_2 -> Net-(U4-BISEN)
- R31 pad 1: /MotorSystem/MotorDriver-3/SENSEI_2 -> Net-(U5-BISEN)
- R32 pad 1: /MotorSystem/MotorDriver-4/SENSEI_2 -> Net-(U6-BISEN)
- R33 pad 1: /MotorSystem/MotorDriver-1/SENSEI_1 -> Net-(U1-AISEN)
- R34 pad 1: /MotorSystem/MotorDriver-2/SENSEI_1 -> Net-(U4-AISEN)
- R35 pad 1: /MotorSystem/MotorDriver-3/SENSEI_1 -> Net-(U5-AISEN)
- R36 pad 1: /MotorSystem/MotorDriver-4/SENSEI_1 -> Net-(U6-AISEN)
- R37 pad 1: /MotorSystem/MotorDriver-1/SENSEI_2 -> Net-(U1-BISEN)
- R37 pad 2: Net-(U10-PA1/ADC_IN1) -> /MotorSystem/MotorDriver-1/SENSEI_2
- R40 pad 1: /MotorSystem/MotorDriver-3/SENSEI_1 -> Net-(U4-AISEN)
- R40 pad 2: Net-(U14-PA0/ADC_IN0) -> /MotorSystem/MotorDriver-2/SENSEI_1
- R41 pad 1: /MotorSystem/MotorDriver-3/SENSEI_2 -> Net-(U4-BISEN)
- R41 pad 2: Net-(U14-PA1/ADC_IN1) -> /MotorSystem/MotorDriver-2/SENSEI_2
- U1 pad 2: Net-(J19-Pin_6) -> Net-(J19-Pin_5)
- U1 pad 3: /MotorSystem/MotorDriver-1/SENSEI_1 -> Net-(U1-AISEN)
- U1 pad 4: Net-(J19-Pin_5) -> Net-(J19-Pin_6)
- U1 pad 6: /MotorSystem/MotorDriver-1/SENSEI_2 -> Net-(U1-BISEN)
- U10 pad 15: /MotorSystem/MotorDriver-2/MOTOR_SIGNAL_2A -> /MotorSystem/MotorDriver-4/MOTOR_SIGNAL_2A
- U10 pad 17: E2A -> E7B
- U10 pad 2: E1A -> E2B
- U10 pad 22: E4A -> E7A
- U10 pad 25: E4B -> E8B
- U10 pad 26: E2B -> E8A
- U10 pad 27: /MotorSystem/MotorDriver-2/MOTOR_SIGNAL_1A -> /MotorSystem/MotorDriver-4/MOTOR_SIGNAL_1A
- U10 pad 28: /MotorSystem/MotorDriver-2/MOTOR_SIGNAL_1B -> /MotorSystem/MotorDriver-4/MOTOR_SIGNAL_1B
- U10 pad 29: E3A -> E1B
- U10 pad 3: E1B -> E2A
- U10 pad 30: E3B -> E1A
- U10 pad 5: /MotorSystem/MotorDriver-2/MOTOR_SIGNAL_2B -> /MotorSystem/MotorDriver-4/MOTOR_SIGNAL_2B
- U10 pad 6: Net-(U10-PA0/ADC_IN0) -> /MotorSystem/MotorDriver-1/SENSEI_1
- U10 pad 7: Net-(U10-PA1/ADC_IN1) -> /MotorSystem/MotorDriver-1/SENSEI_2
- U10 pad 8: Net-(U10-PA2/ADC_IN2) -> /MotorSystem/MotorDriver-4/SENSEI_1
- U10 pad 9: Net-(U10-PA3/ADC_IN3) -> /MotorSystem/MotorDriver-4/SENSEI_2
- U14 pad 15: /MotorSystem/MotorDriver-4/MOTOR_SIGNAL_2A -> /MotorSystem/MotorDriver-2/MOTOR_SIGNAL_2A
- U14 pad 17: E6A -> E3B
- U14 pad 2: E5A -> E6B
- U14 pad 22: E8A -> E3A
- U14 pad 25: E8B -> E4B
- U14 pad 26: E6B -> E4A
- U14 pad 27: /MotorSystem/MotorDriver-4/MOTOR_SIGNAL_1A -> /MotorSystem/MotorDriver-2/MOTOR_SIGNAL_1A
- U14 pad 28: /MotorSystem/MotorDriver-4/MOTOR_SIGNAL_1B -> /MotorSystem/MotorDriver-2/MOTOR_SIGNAL_1B
- U14 pad 29: E7A -> E5B
- U14 pad 3: E5B -> E6A
- U14 pad 30: E7B -> E5A
- U14 pad 5: /MotorSystem/MotorDriver-4/MOTOR_SIGNAL_2B -> /MotorSystem/MotorDriver-2/MOTOR_SIGNAL_2B
- U14 pad 6: Net-(U14-PA0/ADC_IN0) -> /MotorSystem/MotorDriver-3/SENSEI_1
- U14 pad 7: Net-(U14-PA1/ADC_IN1) -> /MotorSystem/MotorDriver-3/SENSEI_2
- U14 pad 8: Net-(U14-PA2/ADC_IN2) -> /MotorSystem/MotorDriver-2/SENSEI_1
- U14 pad 9: Net-(U14-PA3/ADC_IN3) -> /MotorSystem/MotorDriver-2/SENSEI_2
- U2 pad 15: unconnected-(U2-GPIO10-Pad15) -> MOTOR_PYA_SWCLK
- U2 pad 16: unconnected-(U2-GPIO11-Pad16) -> MOTOR_PYA_SWDIO
- U2 pad 17: unconnected-(U2-GPIO12-Pad17) -> MOTOR_PYB_SWCLK
- U2 pad 18: unconnected-(U2-GPIO13-Pad18) -> MOTOR_PYB_SWDIO
- U2 pad 19: unconnected-(U2-GPIO14-Pad19) -> MOTOR_PY_NRST
- U4 pad 2: Net-(J7-Pin_6) -> Net-(J7-Pin_5)
- U4 pad 3: /MotorSystem/MotorDriver-2/SENSEI_1 -> Net-(U4-AISEN)
- U4 pad 4: Net-(J7-Pin_5) -> Net-(J7-Pin_6)
- U4 pad 6: /MotorSystem/MotorDriver-2/SENSEI_2 -> Net-(U4-BISEN)
- U5 pad 2: Net-(J10-Pin_6) -> Net-(J10-Pin_5)
- U5 pad 3: /MotorSystem/MotorDriver-3/SENSEI_1 -> Net-(U5-AISEN)
- U5 pad 4: Net-(J10-Pin_5) -> Net-(J10-Pin_6)
- U5 pad 6: /MotorSystem/MotorDriver-3/SENSEI_2 -> Net-(U5-BISEN)
- U6 pad 2: Net-(J1-Pin_6) -> Net-(J1-Pin_5)
- U6 pad 3: /MotorSystem/MotorDriver-4/SENSEI_1 -> Net-(U6-AISEN)
- U6 pad 4: Net-(J1-Pin_5) -> Net-(J1-Pin_6)
- U6 pad 6: /MotorSystem/MotorDriver-4/SENSEI_2 -> Net-(U6-BISEN)
Routing:
- net Net-(U2-CHIP_PU): track 107.4 -> 0.00 mm, vias 4 -> 0
- net Net-(U2-GPIO0): track 94.7 -> 0.00 mm, vias 4 -> 0
- net Q_SCL: track 83.3 -> 0.00 mm, vias 2 -> 0
- net Q_SDA: track 82.2 -> 0.00 mm, vias 2 -> 0
- net SRV1: track 60.6 -> 0.00 mm, vias 1 -> 0
- net VCC: track 72.8 -> 14.2 mm
- net SRV2: track 56.0 -> 0.00 mm, vias 1 -> 0
- net SRV3: track 53.8 -> 0.00 mm, vias 1 -> 0
- net SF_SDA: track 52.6 -> 1.19 mm, vias 2 -> 1
- net SF_SCL: track 50.7 -> 1.06 mm, vias 2 -> 1
- net SRV4: track 49.0 -> 0.00 mm, vias 1 -> 0
- net GND: track 77.0 -> 30.2 mm, vias 49 -> 10
- net SF_INT2: track 48.4 -> 1.71 mm, vias 2 -> 0
- net GPIO_MISC1: track 45.7 -> 0.00 mm, vias 1 -> 0
- net GPIO_MISC2: track 44.7 -> 0.00 mm, vias 1 -> 0
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- removed copper zone on F.Cu, net GND
- removed copper zone on In1.Cu, net VCC
- removed copper zone on In2.Cu, net VCC
Other:
- board text added: "Alfredo NoU V3.7"
- board text removed: "5K/3K => 0.375*3.3V"
- board text removed: "Alfredo NoU V3.6"
- board text removed: "E1"
- board text removed: "E2"
- board text removed: "E3"
- board text removed: "E4"
- board text removed: "E5"
- board text removed: "E6"
- board text removed: "E7"
- board text removed: "GND"
- board text removed: "RX0"
- board text removed: "SVIN"
- board text removed: "TX0"
- board text removed: "VCC"
