File: NoU3-Lite/NoU3-Lite.kicad_sch (KiCad schematic)
At the start: 71 parts, among them J1 JST SR/SZ, J14 RFANT3216120A5T, J15 Barrel_Jack, J16 VIN, J17 JST SR/SZ, J18 GND, J4 JST SR/SZ, J7 JST SR/SZ, Q20 AO3401A, SW1 reset, SW2 boot, U11 Qwiic1, U15 SY8113BADC, U16 SY8113BADC, U17 USB_C_Receptacle, U18 ServoPorts_2x3, U19 ServoPorts_2x3, U2 ESP32-S3FN8, U3 Crystal_ESP32, U7 ServoPorts_2x3, U8 5.8 ZSPT, U9 USBLC6-2P6

Commit message: first push with NoU3.7 features
Parts:
- U15, U16: symbol NoU265:SY8113BADC -> AlfredoSymbols:SY8113BADC
Changed lines of the file:
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@@
 	)
 	(symbol
-		(lib_id "NoU265:SY8113BADC")
+		(lib_id "AlfredoSymbols:SY8113BADC")
 		(at -76.2 -1.27 0)
 		(unit 1)
@@
 	)
 	(symbol
-		(lib_id "NoU265:SY8113BADC")
+		(lib_id "AlfredoSymbols:SY8113BADC")
 		(at -62.23 -38.1 0)
 		(unit 1)
